Commit message: update

File: assets/ur_description/urdf/ur3_robot_gripper.urdf (robot description, URDF)
Before this commit: robot ur3, 13 links, 12 joints
Joints:
- joint gripper_fixed_joint: limit (none) -> lower=-3.1415926 upper=3.14159263; origin xyz=0 0.24 0.0 rpy=0.0 0.0 3.14159263 -> xyz=0 0.24 0.0 rpy=0.0 3.1415926 3.14159263
- joint shaft_fixed_joint: origin xyz=0 0.0 0.0 rpy=0.0 1.57 3.14159263 -> xyz=0 0.0 0.0 rpy=0.0 -1.57 3.14159263

Commit message: update assembly

File: assets/ur_description/urdf/ur3_robot_gripper.urdf (robot description, URDF)
Before this commit: robot ur3, 13 links, 12 joints
Joints:
- joint shaft_fixed_joint: origin xyz=0 0.0 0.0 rpy=0.0 -1.57 3.14159263 -> xyz=0 0.0 0.11 rpy=0.0 -1.57 3.14159263
