Commit message: add ur5_package

File: assets/ur_robotics/ur5_gripper/ur5_gripper_origin.urdf (robot description, URDF)
Before this commit: robot ur5, 21 links, 20 joints
Joints:
- joint robotiq_85_left_finger_tip_joint: type fixed -> continuous
- joint robotiq_85_left_inner_knuckle_joint: type fixed -> continuous
- joint robotiq_85_left_knuckle_joint: type fixed -> revolute
- joint robotiq_85_right_finger_tip_joint: type fixed -> continuous
- joint robotiq_85_right_inner_knuckle_joint: type fixed -> continuous
- joint robotiq_85_right_knuckle_joint: type fixed -> continuous

File: assets/ur_robotics/ur5_gripper/ur5_gripper_shaft.urdf (robot description, URDF)
Before this commit: robot ur5, 21 links, 20 joints
Links:
- added link shaft_link, mass 0.12491; collision mesh filename=shaft/meshes/base_link.STL; visual mesh filename=shaft/meshes/base_link.STL
Joints:
- added joint shaft_joint: type fixed, parent wrist_3_link, child shaft_link, origin xyz=-0.0 0.26 -0.06 rpy=1.57 1.57 0.0

Commit message: add separate

File: assets/ur_robotics/ur5_gripper/ur5_gripper_origin.urdf (robot description, URDF)
Before this commit: robot ur5, 21 links, 20 joints
Links:
- added link gripper_link, mass 1; collision mesh filename=package://meshes_gripper/toolMount.STL; visual mesh filename=package://meshes_gripper/toolMount.STL
- added link shaft_link, mass 1; collision mesh filename=package://meshes_gripper/shaft.STL; visual mesh filename=package://meshes_gripper/shaft.STL
Joints:
- added joint gripper_fixed_joint: type revolute, parent wrist_3_link, child gripper_link, origin xyz=0 0.24 0.0 rpy=0.0 3.1415926 3.14159263, axis 0 1 0, limit lower=-3.1415926 upper=3.14159263
- added joint shaft_fixed_joint: type fixed, parent gripper_link, child shaft_link, origin xyz=0 0.0 0.11 rpy=0.0 -1.57 3.14159263

File: assets/ur_robotics/ur5e/ur5e.urdf (robot description, URDF)
Before this commit: robot ur5e, 11 links, 10 joints
Links:
- added link gripper_link, mass 1; collision mesh filename=package://meshes_gripper/toolMount.STL; visual mesh filename=package://meshes_gripper/toolMount.STL
- added link shaft_link, mass 1; collision mesh filename=package://meshes_gripper/shaft.STL; visual mesh filename=package://meshes_gripper/shaft.STL
Joints:
- added joint gripper_fixed_joint: type revolute, parent wrist_3_link, child gripper_link, origin xyz=0 0.24 0.0 rpy=0.0 3.1415926 3.14159263, axis 0 1 0, limit lower=-3.1415926 upper=3.14159263
- added joint shaft_fixed_joint: type fixed, parent gripper_link, child shaft_link, origin xyz=0 0.0 0.11 rpy=0.0 -1.57 3.14159263
- joint shoulder_pan_joint: origin xyz=0.0 0.0 0.163 rpy=0.0 -1.57 0.0 -> xyz=0.0 0.0 0.163 rpy=0.0 -0 0.0
